Commit message: updates

File: rso2_ws/install/my_robot_description/share/my_robot_description/urdf/common_properties.xacro (robot description, xacro)
@@ -1 +1,44 @@
-/home/marco/projects/ros/rso2_ws/src/my_robot_description/urdf/common_properties.xacro
+<?xml version= "1.0"?>
+<robot  xmlns:xacro="http://www.ros.org/wiki/xacro">
+    <material name="blue">
+        <color rgba="0 0 0.5 1"/>
+    </material>
+    <material name="green">
+        <color rgba="0 0.5 0 1"/>
+    </material>
+    <material name="grey">
+        <color rgba="0.5 0.5 0.5 1"/>
+    </material>
+    <material name="red">
+        <color rgba="0.5 0 0 1"/>
+    </material>
+    <xacro:macro name = "box_inertia"   params = "m l w h xyz rpy">
+        <inertial>
+            <origin xyz = "${xyz}" rpy="${rpy}"/>
+            <mass value = "${m}"/>
+            <inertia ixx = "${(m/12)*(h*h + l*l)}" ixy = "0" ixz = "0"
+            iyy = "${(m/12)*(w*w + l*l)}" iyz = "0"
+            izz = "${(m/12)*(w*w + h*h)}"
+            />
+        </inertial>
+    </xacro:macro>
+    <xacro:macro name = "sphere_inertia"   params = "m r xyz rpy">
+        <inertial>
+            <origin xyz = "${xyz}" rpy="${rpy}"/>
+            <mass value = "${m}"/>
+            <inertia ixx = "${m*(2/5)*(r*r)}" ixy = "0" ixz = "0"
+            iyy = "${m*(2/5)*(r*r)}" iyz = "0"
+            izz = "${m*(2/5)*(r*r)}"
+            />
+        </inertial>
+    </xacro:macro>
+      <xacro:macro name = "cilinder_inertia"   params = "m r h xyz rpy">
+        <inertial>
+            <origin xyz = "${xyz}" rpy="${rpy}"/>
+            <mass value = "${m}"/>
+            <inertia ixx = "${(m/12)*(3*r*r + h*h )}" ixy = "0" ixz = "0"
+            iyy = "${(m/12)*(3*r*r + h*h)}" iyz = "0"
+            izz ="${(m/2)*(r*r)}" />
+        </inertial>
+    </xacro:macro>
+</robot>

File: rso2_ws/install/my_robot_description/share/my_robot_description/urdf/drone.urdf.xacro (robot description, xacro)
@@ -1 +1,113 @@
-/home/marco/projects/ros/rso2_ws/src/my_robot_description/urdf/drone.urdf.xacro
+<?xml version="1.0"?>
+   <robot name="drone">
+     <link name="base_link">
+       <visual>
+		 <origin xyz="0 0 0" rpy="0 0 0" />
+         <geometry>
+           <box size="0.4 0.2 0.04"/>
+         </geometry>
+       </visual>
+       <collision>
+		  <origin xyz="0 0 0" rpy="0 0 0" />
+          <geometry>
+            <box size="0.4 0.04 0.04"/>
+          </geometry>
+        </collision>
+        <!--<inertial>
+           <mass value="0.3"/>
+           <inertia ixx="1.0" ixy="0.0" ixz="0.0" iyy="1.0" iyz="0.0" izz="1.0"/>
+         </inertial>-->
+     </link>
+     <link name="FL">
+       <visual>
+		 <origin xyz="0.16 0.13 0" rpy="0 0 0" />
+         <geometry>
+            <cylinder length="0.03" radius="0.13"/>
+         </geometry>
+       </visual>
+       <collision>
+          <origin xyz="0.16 0.13 0" rpy="0 0 0" />
+          <geometry>
+            <cylinder length="0.03" radius="0.13"/>
+          </geometry>
+        </collision>
+        <inertial>
+           <mass value="0.2"/>
+           <inertia ixx="1.0" ixy="0.0" ixz="0.0" iyy="1.0" iyz="0.0" izz="1.0"/>
+         </inertial>
+     </link>
+     <link name="FR">
+       <visual>
+		 <origin xyz="0.16 -0.13 0" rpy="0 0 0" />
+         <geometry>
+            <cylinder length="0.03" radius="0.13"/>
+         </geometry>
+       </visual>
+       <collision>
+          <origin xyz="0.16 -0.13 0" rpy="0 0 0" />
+          <geometry>
+            <cylinder length="0.03" radius="0.13"/>
+          </geometry>
+        </collision>
+        <inertial>
+           <mass value="0.2"/>
+           <inertia ixx="1.0" ixy="0.0" ixz="0.0" iyy="1.0" iyz="0.0" izz="1.0"/>
+         </inertial>
+     </link>
+     <link name="BL">
+       <visual>
+		 <origin xyz="-0.09 0.13 0" rpy="0 0 0" />
+         <geometry>
+            <cylinder length="0.03" radius="0.13"/>
+         </geometry>
+       </visual>
+       <collision>
+          <origin xyz="-0.09 0.13 0" rpy="0 0 0" />
+          <geometry>
+            <cylinder length="0.03" radius="0.13"/>
+          </geometry>
+        </collision>
+        <inertial>
+           <mass value="0.2"/>
+           <inertia ixx="1.0" ixy="0.0" ixz="0.0" iyy="1.0" iyz="0.0" izz="1.0"/>
+         </inertial>
+     </link>
+     <link name="BR">
+       <visual>
+		 <origin xyz="-0.09 -0.13 0" rpy="0 0 0" />
+         <geometry>
+            <cylinder length="0.03" radius="0.13"/>
+         </geometry>
+       </visual>
+       <collision>
+          <origin xyz="-0.09 -0.13 0" rpy="0 0 0" />
+          <geometry>
+            <cylinder length="0.03" radius="0.13"/>
+          </geometry>
+        </collision>
+        <inertial>
+           <mass value="0.2"/>
+           <inertia ixx="1.0" ixy="0.0" ixz="0.0" iyy="1.0" iyz="0.0" izz="1.0"/>
+         </inertial>
+     </link>
+     <joint name="base_to_FL" type="fixed">
+       <parent link="base_link"/>
+       <child link="FL"/>
+     </joint>
+     <joint name="base_to_FR" type="fixed">
+       <parent link="base_link"/>
+       <child link="FR"/>
+     </joint>
+     <joint name="base_to_BL" type="fixed">
+       <parent link="base_link"/>
+       <child link="BL"/>
+     </joint>
+     <joint name="base_to_BR" type="fixed">
+       <parent link="base_link"/>
+       <child link="BR"/>
+     </joint>
+     <gazebo reference="base_link">
+       <material>Gazebo/Blue</material>
+       <turnGravityOff>true</turnGravityOff>
+     </gazebo>
+   </robot>

File: rso2_ws/install/my_robot_description/share/my_robot_description/urdf/mobile_base.xacro (robot description, xacro)
@@ -1 +1,87 @@
-/home/marco/projects/ros/rso2_ws/src/my_robot_description/urdf/mobile_base.xacro
+<?xml version= "1.0"?>
+<robot  xmlns:xacro="http://www.ros.org/wiki/xacro">
+    <xacro:property name = "base_length" value = "0.6"/>
+    <xacro:property name = "base_width" value =  "0.4"/>
+    <xacro:property name = "base_height" value =  "0.2"/>
+    <xacro:property name = "wheel_radius" value = "0.1"/>
+    <xacro:property name = "wheel_length" value = "0.05"/>
+    <link name= "base_footprint"/>
+    <link name="base_link">
+        <visual>
+            <geometry>
+                <box size="${base_length} ${base_width} ${base_height}"/>
+            </geometry>
+            <origin xyz="0 0 0.1" rpy="0 0 0"/>
+            <material name= "grey" />
+        </visual>
+        <collision>
+             <geometry>
+                <box size="${base_length} ${base_width} ${base_height}"/>
+            </geometry>
+            <origin xyz="0 0 0.1" rpy="0 0 0"/>
+        </collision>
+        <xacro:box_inertia m ="5.0"  l = "${base_length}" w = "${base_width}"
+        h= "${base_height}" xyz = "0 0 0.1" rpy = "0 0 0"/>
+    </link>
+    <xacro:macro name= "wheel_link" params = "prefix">
+        <link name= "${prefix}_wheel_link">
+            <visual>
+                <geometry>
+                    <cylinder radius= "${wheel_radius}" length="${wheel_length}"/>
+                </geometry>
+                <origin xyz= "0 0 0" rpy="${pi/2.0} 0 0"/>
+                <material   name="red" />
+            </visual>
+        <collision>
+            <geometry>
+                <cylinder radius= "${wheel_radius}" length="${wheel_length}"/>
+            </geometry>
+            <origin xyz= "0 0 0" rpy="${pi/2.0} 0 0"/>
+        </collision>
+        </link>
+        <xacro:cilinder_inertia m =  "0.5" r= "${wheel_radius}"
+        h= "${wheel_length}" xyz =  "0 0 0" rpy="${pi/2.0} 0 0"/>
+    </xacro:macro>
+    <xacro:wheel_link prefix="right"/>
+    <xacro:wheel_link prefix="left"/>
+   <link name= "middle_wheel_link">
+        <visual>
+            <geometry>
+                <sphere radius= "${wheel_radius/2.0}" />
+            </geometry>
+            <origin xyz= "0 0 0" rpy="0 0 0"/>
+            <material   name="red" />
+        </visual>
+        <collision>
+            <geometry>
+                <sphere radius= "${wheel_radius/2.0}" />
+            </geometry>
+            <origin xyz= "0 0 0" rpy="0 0 0"/>
+        </collision>
+        <xacro:sphere_inertia m = "1.0" r = "${wheel_radius/2.0}"
+        xyz = "0 0 0" rpy= "0 0 0"/>
+   </link>
+   <joint name= "base_joint" type= "fixed">
+        <parent link= "base_footprint"/>
+        <child link = "base_link"/>
+        <origin xyz= "0 0 0.1" rpy= "0 0 0"/>
+   </joint>
+    <joint name= "base_right_wheel_joint" type="continuous">
+            <parent link=  "base_link" />
+            <child link = "right_wheel_link" />
+            <origin xyz = "${-base_length/4.0} ${-(base_width + wheel_length)/2.0} 0" rpy="0 0 0" />
+            <axis xyz="0 1 0"/>
+    </joint>
+    <joint name= "base_left_wheel_joint" type="continuous">
+            <parent link=  "base_link" />
+            <child link = "left_wheel_link" />
+            <origin xyz = "${-base_length/4.0} ${(base_width + wheel_length)/2.0} 0" rpy="0 0 0" />
+            <axis xyz="0 1 0"/>
+    </joint>
+     <joint name= "base_middle_wheel_joint" type="fixed">
+            <parent link=  "base_link" />
+            <child link = "middle_wheel_link" />
+            <origin xyz = "${base_length/3.0} 0 ${-wheel_radius/2.0}" rpy="0 0 0" />
+            <axis xyz="0 1 0"/>
+    </joint>
+</robot>

File: rso2_ws/install/my_robot_description/share/my_robot_description/urdf/my_robot.urdf.xacro (robot description, xacro)
@@ -1 +1,5 @@
-/home/marco/projects/ros/rso2_ws/src/my_robot_description/urdf/my_robot.urdf.xacro
+<?xml version="1.0"?>
+<robot name="my_robot" xmlns:xacro="http://www.ros.org/wiki/xacro">
+    <xacro:include filename="common_properties.xacro" />
+    <xacro:include filename="mobile_base.xacro" />
+</robot>

File: rso2_ws/src/my_robot_description/urdf/my_robot.urdf.xacro (robot description, xacro)
@@ -1,5 +1,5 @@
-<?xml version= "1.0"?>
+<?xml version="1.0"?>
 <robot name="my_robot" xmlns:xacro="http://www.ros.org/wiki/xacro">
-    <xacro:include  filename= "common_properties.xacro"/>
-    <xacro:include  filename  ="mobile_base.xacro"/>
+    <xacro:include filename="common_properties.xacro" />
+    <xacro:include filename="mobile_base.xacro" />
 </robot>
