Commit message: updates

File: rso2_ws/install/my_robot_description/share/my_robot_description/urdf/mobile_base.xacro (robot description, xacro)
@@ -35,11 +35,11 @@
         <collision>
             <geometry>
-                <cylinder radius= "${wheel_radius}" length="${wheel_length}"/>
+                <sphere radius= "${wheel_radius}" />
             </geometry>
-            <origin xyz= "0 0 0" rpy="${pi/2.0} 0 0"/>
+             <origin xyz= "0 0 0" rpy="0 0 0"/>
         </collision>
+          <xacro:cilinder_inertia m =  "0.5" r= "${wheel_radius}"
+          h= "${wheel_length}" xyz =  "0 0 0" rpy="${pi/2.0} 0 0"/>
         </link>
-        <xacro:cilinder_inertia m =  "0.5" r= "${wheel_radius}"
-        h= "${wheel_length}" xyz =  "0 0 0" rpy="${pi/2.0} 0 0"/>
     </xacro:macro>
     <xacro:wheel_link prefix="right"/>

File: rso2_ws/install/my_robot_description/share/my_robot_description/urdf/my_robot.urdf.xacro (robot description, xacro)
@@ -3,3 +3,4 @@
     <xacro:include filename="common_properties.xacro" />
     <xacro:include filename="mobile_base.xacro" />
+    <xacro:include filename="mobile_base_gazebo.xacro" />
 </robot>

File: rso2_ws/src/my_robot_description/urdf/mobile_base.xacro (robot description, xacro)
@@ -35,11 +35,11 @@
         <collision>
             <geometry>
-                <cylinder radius= "${wheel_radius}" length="${wheel_length}"/>
+                <sphere radius= "${wheel_radius}" />
             </geometry>
-            <origin xyz= "0 0 0" rpy="${pi/2.0} 0 0"/>
+             <origin xyz= "0 0 0" rpy="0 0 0"/>
         </collision>
+          <xacro:cilinder_inertia m =  "0.5" r= "${wheel_radius}"
+          h= "${wheel_length}" xyz =  "0 0 0" rpy="${pi/2.0} 0 0"/>
         </link>
-        <xacro:cilinder_inertia m =  "0.5" r= "${wheel_radius}"
-        h= "${wheel_length}" xyz =  "0 0 0" rpy="${pi/2.0} 0 0"/>
     </xacro:macro>
     <xacro:wheel_link prefix="right"/>
