Commit message: updates

File: rso2_ws/src/my_robot_description/urdf/common_properties.xacro (robot description, xacro)
@@ -1,43 +1,35 @@
-<?xml version= "1.0"?>
-<robot  xmlns:xacro="http://www.ros.org/wiki/xacro">
+<?xml version="1.0"?>
+<robot xmlns:xacro="http://www.ros.org/wiki/xacro">
     <material name="blue">
-        <color rgba="0 0 0.5 1"/>
-    </material>
-    <material name="green">
-        <color rgba="0 0.5 0 1"/>
+        <color rgba="0 0 0.5 1" />
     </material>
     <material name="grey">
-        <color rgba="0.5 0.5 0.5 1"/>
+        <color rgba="0.5 0.5 0.5 1" />
     </material>
-    <material name="red">
-        <color rgba="0.5 0 0 1"/>
-    </material>
-    <xacro:macro name = "box_inertia"   params = "m l w h xyz rpy">
+    <xacro:macro name="box_inertia" params="m x y z o_xyz o_rpy">
         <inertial>
-            <origin xyz = "${xyz}" rpy="${rpy}"/>
-            <mass value = "${m}"/>
-            <inertia ixx = "${(m/12)*(h*h + l*l)}" ixy = "0" ixz = "0"
-            iyy = "${(m/12)*(w*w + l*l)}" iyz = "0"
-            izz = "${(m/12)*(w*w + h*h)}"
-            />
+            <mass value="${m}" />
+            <origin xyz="${o_xyz}" rpy="${o_rpy}" />
+            <inertia ixx="${(m/12) * (y*y + z*z)}" ixy="0" ixz="0"
+                     iyy="${(m/12) * (x*x + z*z)}" iyz="0"
+                     izz="${(m/12) * (x*x + y*y)}" />
         </inertial>
     </xacro:macro>
-    <xacro:macro name = "sphere_inertia"   params = "m r xyz rpy">
+    <xacro:macro name="cylinder_inertia" params="m r l o_xyz o_rpy">
         <inertial>
-            <origin xyz = "${xyz}" rpy="${rpy}"/>
-            <mass value = "${m}"/>
-            <inertia ixx = "${m*(2/5)*(r*r)}" ixy = "0" ixz = "0"
-            iyy = "${m*(2/5)*(r*r)}" iyz = "0"
-            izz = "${m*(2/5)*(r*r)}"
-            />
+            <mass value="${m}" />
+            <origin xyz="${o_xyz}" rpy="${o_rpy}" />
+            <inertia ixx="${(m/12) * (3*r*r + l*l)}" ixy="0" ixz="0"
+                     iyy="${(m/12) * (3*r*r + l*l)}" iyz="0"
+                     izz="${(m/2) * (r*r)}" />
         </inertial>
     </xacro:macro>
-      <xacro:macro name = "cilinder_inertia"   params = "m r h xyz rpy">
+    <xacro:macro name="sphere_inertia" params="m r o_xyz o_rpy">
         <inertial>
-            <origin xyz = "${xyz}" rpy="${rpy}"/>
-            <mass value = "${m}"/>
-            <inertia ixx = "${(m/12)*(3*r*r + h*h )}" ixy = "0" ixz = "0"
-            iyy = "${(m/12)*(3*r*r + h*h)}" iyz = "0"
-            izz ="${(m/2)*(r*r)}" />
+            <mass value="${m}" />
+            <origin xyz="${o_xyz}" rpy="${o_rpy}" />
+            <inertia ixx="${(2/5) * m * r * r}" ixy="0" ixz="0"
+                     iyy="${(2/5) * m * r * r}" iyz="0"
+                     izz="${(2/5) * m * r * r}" />
         </inertial>
     </xacro:macro>

File: rso2_ws/src/my_robot_description/urdf/mobile_base.xacro (robot description, xacro)
@@ -1,87 +1,134 @@
-<?xml version= "1.0"?>
-<robot  xmlns:xacro="http://www.ros.org/wiki/xacro">
-    <xacro:property name = "base_length" value = "0.6"/>
-    <xacro:property name = "base_width" value =  "0.4"/>
-    <xacro:property name = "base_height" value =  "0.2"/>
-    <xacro:property name = "wheel_radius" value = "0.1"/>
-    <xacro:property name = "wheel_length" value = "0.05"/>
-    <link name= "base_footprint"/>
-    <link name="base_link">
-        <visual>
-            <geometry>
-                <box size="${base_length} ${base_width} ${base_height}"/>
-            </geometry>
-            <origin xyz="0 0 0.1" rpy="0 0 0"/>
-            <material name= "grey" />
-        </visual>
-        <collision>
-             <geometry>
-                <box size="${base_length} ${base_width} ${base_height}"/>
-            </geometry>
-            <origin xyz="0 0 0.1" rpy="0 0 0"/>
-        </collision>
-        <xacro:box_inertia m ="5.0"  l = "${base_length}" w = "${base_width}"
-        h= "${base_height}" xyz = "0 0 0.1" rpy = "0 0 0"/>
+<?xml version="1.0"?>
+<robot xmlns:xacro="http://www.ros.org/wiki/xacro">
+  <!-- Properties -->
+  <xacro:property name="base_length" value="0.6" />
+  <xacro:property name="base_width" value="0.4" />
+  <xacro:property name="base_height" value="0.2" />
+  <xacro:property name="wheel_radius" value="0.1" />
+  <xacro:property name="wheel_length" value="0.05" />
+  <!-- Materials -->
+  <material name="blue"><color rgba="0 0 0.5 1"/></material>
+  <material name="green"><color rgba="0 0.5 0 1"/></material>
+  <material name="grey"><color rgba="0.5 0.5 0.5 1"/></material>
+  <material name="red"><color rgba="0.5 0 0 1"/></material>
+  <!-- Macros -->
+  <xacro:macro name="box_inertia" params="m l w h xyz rpy">
+    <inertial>
+      <origin xyz="${xyz}" rpy="${rpy}"/>
+      <mass value="${m}"/>
+      <inertia ixx="${(m/12)*(h*h + l*l)}" ixy="0" ixz="0"
+               iyy="${(m/12)*(w*w + l*l)}" iyz="0"
+               izz="${(m/12)*(w*w + h*h)}"/>
+    </inertial>
+  </xacro:macro>
+  <xacro:macro name="sphere_inertia" params="m r xyz rpy">
+    <inertial>
+      <origin xyz="${xyz}" rpy="${rpy}"/>
+      <mass value="${m}"/>
+      <inertia ixx="${m*(2/5)*(r*r)}" ixy="0" ixz="0"
+               iyy="${m*(2/5)*(r*r)}" iyz="0"
+               izz="${m*(2/5)*(r*r)}"/>
+    </inertial>
+  </xacro:macro>
+  <xacro:macro name="cylinder_inertia" params="m r l xyz rpy">
+    <inertial>
+      <origin xyz="${xyz}" rpy="${rpy}"/>
+      <mass value="${m}"/>
+      <inertia ixx="${(m/12)*(3*r*r + l*l)}" ixy="0" ixz="0"
+               iyy="${(m/12)*(3*r*r + l*l)}" iyz="0"
+               izz="${(m/2)*(r*r)}"/>
+    </inertial>
+  </xacro:macro>
+  <!-- Robot Links -->
+  <link name="base_footprint"/>
+  <link name="base_link">
+    <visual>
+      <geometry>
+        <box size="${base_length} ${base_width} ${base_height}" />
+      </geometry>
+      <origin xyz="0 0 ${base_height / 2.0}" rpy="0 0 0" />
+      <material name="blue"/>
+    </visual>
+    <collision>
+      <geometry>
+        <box size="${base_length} ${base_width} ${base_height}" />
+      </geometry>
+      <origin xyz="0 0 ${base_height / 2.0}" rpy="0 0 0" />
+    </collision>
+    <xacro:box_inertia m="5.0"
+                       l="${base_length}"
+                       w="${base_width}"
+                       h="${base_height}"
+                       xyz="0 0 ${base_height / 2.0}"
+                       rpy="0 0 0" />
+  </link>
+  <!-- Wheel Macro -->
+  <xacro:macro name="wheel_link" params="prefix">
+    <link name="${prefix}_wheel_link">
+      <visual>
+        <geometry>
+          <cylinder radius="${wheel_radius}" length="${wheel_length}" />
+        </geometry>
+        <origin xyz="0 0 0" rpy="${pi / 2.0} 0 0" />
+        <material name="grey" />
+      </visual>
+      <collision>
+        <geometry>
+          <sphere radius="${wheel_radius}" />
+        </geometry>
+        <origin xyz="0 0 0" rpy="0 0 0" />
+      </collision>
+      <xacro:cylinder_inertia m="1.0"
+                              r="${wheel_radius}"
+                              l="${wheel_length}"
+                              xyz="0 0 0"
+                              rpy="${pi / 2.0} 0 0" />
     </link>
-    <xacro:macro name= "wheel_link" params = "prefix">
-        <link name= "${prefix}_wheel_link">
-            <visual>
-                <geometry>
-                    <cylinder radius= "${wheel_radius}" length="${wheel_length}"/>
-                </geometry>
-                <origin xyz= "0 0 0" rpy="${pi/2.0} 0 0"/>
-                <material   name="red" />
-            </visual>
-        <collision>
-            <geometry>
-                <sphere radius= "${wheel_radius}" />
-            </geometry>
-             <origin xyz= "0 0 0" rpy="0 0 0"/>
-        </collision>
-          <xacro:cilinder_inertia m =  "0.5" r= "${wheel_radius}"
-          h= "${wheel_length}" xyz =  "0 0 0" rpy="${pi/2.0} 0 0"/>
-        </link>
-    </xacro:macro>
-    <xacro:wheel_link prefix="right"/>
-    <xacro:wheel_link prefix="left"/>
-   <link name= "middle_wheel_link">
-        <visual>
-            <geometry>
-                <sphere radius= "${wheel_radius/2.0}" />
-            </geometry>
-            <origin xyz= "0 0 0" rpy="0 0 0"/>
-            <material   name="red" />
-        </visual>
-        <collision>
-            <geometry>
-                <sphere radius= "${wheel_radius/2.0}" />
-            </geometry>
-            <origin xyz= "0 0 0" rpy="0 0 0"/>
-        </collision>
-        <xacro:sphere_inertia m = "1.0" r = "${wheel_radius/2.0}"
-        xyz = "0 0 0" rpy= "0 0 0"/>
-   </link>
-   <joint name= "base_joint" type= "fixed">
-        <parent link= "base_footprint"/>
-        <child link = "base_link"/>
-        <origin xyz= "0 0 0.1" rpy= "0 0 0"/>
-   </joint>
-    <joint name= "base_right_wheel_joint" type="continuous">
-            <parent link=  "base_link" />
-            <child link = "right_wheel_link" />
-            <origin xyz = "${-base_length/4.0} ${-(base_width + wheel_length)/2.0} 0" rpy="0 0 0" />
-            <axis xyz="0 1 0"/>
-    </joint>
-    <joint name= "base_left_wheel_joint" type="continuous">
-            <parent link=  "base_link" />
-            <child link = "left_wheel_link" />
-            <origin xyz = "${-base_length/4.0} ${(base_width + wheel_length)/2.0} 0" rpy="0 0 0" />
-            <axis xyz="0 1 0"/>
-    </joint>
-     <joint name= "base_middle_wheel_joint" type="fixed">
-            <parent link=  "base_link" />
-            <child link = "middle_wheel_link" />
-            <origin xyz = "${base_length/3.0} 0 ${-wheel_radius/2.0}" rpy="0 0 0" />
-            <axis xyz="0 1 0"/>
-    </joint>
+  </xacro:macro>
+  <!-- Instantiate Wheels -->
+  <xacro:wheel_link prefix="right" />
+  <xacro:wheel_link prefix="left" />
+  <!-- Extra Front Sphere -->
+  <link name="_wheel_link">
+    <visual>
+      <geometry>
+        <sphere radius="${wheel_radius / 2.0}" />
+      </geometry>
+      <origin xyz="0 0 0" rpy="0 0 0" />
+      <material name="grey" />
+    </visual>
+    <collision>
+      <geometry>
+        <sphere radius="${wheel_radius / 2.0}" />
+      </geometry>
+      <origin xyz="0 0 0" rpy="0 0 0" />
+    </collision>
+    <xacro:sphere_inertia m="0.5"
+                          r="${wheel_radius / 2.0}"
+                          xyz="0 0 0"
+                          rpy="0 0 0" />
+  </link>
+  <!-- Joints -->
+  <joint name="base_joint" type="fixed">
+    <parent link="base_footprint" />
+    <child link="base_link" />
+    <origin xyz="0 0 ${wheel_radius}" rpy="0 0 0" />
+  </joint>
+  <joint name="base_right_wheel_joint" type="continuous">
+    <parent link="base_link" />
+    <child link="right_wheel_link" />
+    <origin xyz="${-base_length / 4.0} ${-(base_width + wheel_length) / 2.0} 0" rpy="0 0 0" />
+    <axis xyz="0 1 0" />
+  </joint>
+  <joint name="base_left_wheel_joint" type="continuous">
+    <parent link="base_link" />
+    <child link="left_wheel_link" />
+    <origin xyz="${-base_length / 4.0} ${(base_width + wheel_length) / 2.0} 0" rpy="0 0 0" />
+    <axis xyz="0 1 0" />
+  </joint>
+  <joint name="base__wheel_joint" type="fixed">
+    <parent link="base_link" />
+    <child link="_wheel_link" />
+    <origin xyz="${base_length / 3.0} 0 ${-wheel_radius / 2.0}" rpy="0 0 0" />
+  </joint>
 </robot>

File: rso2_ws/src/my_robot_description/urdf/my_robot.urdf.xacro (robot description, xacro)
@@ -4,3 +4,4 @@
     <xacro:include filename="mobile_base.xacro" />
     <xacro:include filename="mobile_base_gazebo.xacro" />
+    <xacro:include filename="camera.xacro" />
 </robot>
